Commit message: montage de la navette + redefinition du modele urdf (ajout joints continus et ajout roue )

File: aip_gazebo/models/shuttle.urdf.xacro (robot description, xacro)
@@ -47,48 +47,111 @@
   <link name="cylinder1">
     <collision>
-      <origin xyz="0 0 0.065" rpy="0 0 0"/>
       <geometry>
         <cylinder radius="0.05" length="0.07"/>
       </geometry>
     </collision>
-    <inertial>
-      <origin xyz="0 0 0.01" rpy="0 0 0"/>
-      <mass value="0"/>
-      <inertia
-        ixx="0.01" ixy="0" ixz="0"
-        iyy="0.02" iyz="0"
-        izz="0.001"/>
-    </inertial>
-  </link>
+      <inertial>
+        <origin rpy="0 0 0" xyz="0 0 0" />
+        <mass value="0.000010000" />
+        <inertia ixx="0.000000010" ixy="0.000000000" ixz="0.000000000" iyy="0.000000010" iyz="0.000000000" izz="0.000000013"/>
+      </inertial>
+    </link>
   <link name="cylinder2">
     <collision>
-      <origin xyz="0 0 0.065" rpy="0 0 0"/>
       <geometry>
         <cylinder radius="0.05" length="0.07"/>
       </geometry>
     </collision>
+      <inertial>
+        <origin rpy="0 0 0" xyz="0 0 0" />
+        <mass value="0.000010000" />
+        <inertia ixx="0.000000010" ixy="0.000000000" ixz="0.000000000" iyy="0.000000010" iyz="0.000000000" izz="0.000000013"/>
+      </inertial>
+    </link>
+  <link name="head_plate">
+    <visual>
+      <geometry>
+        <box size="0.03 0.05 0.01" />
+      </geometry>
+    </visual>
+    <collision>
+      <geometry>
+        <box size="0.03 0.05 0.01" />
+      </geometry>
+    </collision>
     <inertial>
-      <origin xyz="0 0 0.01" rpy="0 0 0"/>
-      <mass value="0"/>
-      <inertia
-        ixx="0.01" ixy="0" ixz="0"
-        iyy="0.02" iyz="0"
-        izz="0.001"/>
+      <origin rpy="0 0 0" xyz="0 0 0" />
+      <mass value="0.000010000" />
+      <inertia ixx="0.000000002" ixy="0.000000000" ixz="0.000000000" iyy="0.000000001" iyz="0.000000000" izz="0.000000003"/>
     </inertial>
-  </link>
-  <joint name="base_joint" type="fixed">
-    <parent link="base_link"/>
-    <child link="body"/>
-    <origin xyz="0 0 0" rpy="0 0 0"/>
+        </link>
+  <link name="free_wheel_1">
+    <visual>
+      <geometry>
+        <cylinder radius="0.01" length="0.02"/>
+      </geometry>
+    </visual>
+    <collision>
+      <geometry>
+        <cylinder radius="0.01" length="0.02"/>
+      </geometry>
+    </collision>
+    <inertial>
+      <origin rpy="0 0 0" xyz="0 0 0" />
+      <mass value="0.000010000" />
+      <inertia ixx="0.000000001" ixy="0.000000000" ixz="0.000000000" iyy="0.000000001" iyz="0.000000000" izz="0.000000001"/>
+    </inertial>
+      </link>
+  <link name="free_wheel_2">
+    <visual>
+      <geometry>
+        <cylinder radius="0.01" length="0.02"/>
+      </geometry>
+    </visual>
+    <collision>
+      <geometry>
+        <cylinder radius="0.01" length="0.02"/>
+      </geometry>
+    </collision>
+    <inertial>
+      <origin rpy="0 0 0" xyz="0 0 0" />
+      <mass value="0.000010000" />
+      <inertia ixx="0.000000001" ixy="0.000000000" ixz="0.000000000" iyy="0.000000001" iyz="0.000000000" izz="0.000000001"/>
+    </inertial>
+    </link>
+<joint name="base_joint" type="fixed">
+  <parent link="base_link"/>
+  <child link="body"/>
+  <origin xyz="0 0 0" rpy="0 0 0"/>
 </joint>
-<joint name="cylinder1_joint" type="fixed">
+<joint name="cylinder1_joint" type="continuous">
+<parent link="body"/>
+<child link="cylinder1"/>
+<axis xyz="0 0 1"/>
+<origin xyz="0 0.07 0.065" rpy="0 0 0"/>
+</joint>
+<joint name="cylinder2_joint" type="continuous">
+<parent link="body"/>
+<child link="cylinder2"/>
+<axis xyz="0 0 1"/>
+<origin xyz="0 -0.07 0.065" rpy="0 0 0"/>
+</joint>
+<joint name="free_plate" type="fixed">
   <parent link="body"/>
-  <child link="cylinder1"/>
-  <origin xyz="0 0.07 0" rpy="0 0 0"/>
+  <child link="head_plate"/>
+  <axis xyz="0 0 1"/>
+  <origin xyz="0.3 0 0.11" rpy="0 0 0"/>
 </joint>
-<joint name="cylinder2_joint" type="fixed">
-  <parent link="body"/>
-  <child link="cylinder2"/>
-  <origin xyz="0 -0.07 0" rpy="0 0 0"/>
+<joint name="free_wheel_1_joint" type="fixed">
+  <parent link="head_plate"/>
+  <child link="free_wheel_1"/>
+  <axis xyz="0 0 1"/>
+  <origin xyz="0 0.03 -0.01" rpy="0 0 0"/>
+</joint>
+<joint name="free_wheel_2_joint" type="continuous">
+  <parent link="head_plate"/>
+  <child link="free_wheel_2"/>
+  <axis xyz="0 0 1"/>
+  <origin xyz="0 -0.03 -0.01" rpy="0 0 0"/>
 </joint>
 <gazebo reference="body">

Commit message: adding topics and motors to control the velocity of the motors of the shuttles + controlling N shuttles separately

File: aip_gazebo/models/shuttle.urdf.xacro (robot description, xacro)
@@ -28,5 +28,5 @@
             <max_vel>0.1</max_vel>
             <soft_cfm>0.8</soft_cfm>
-            <soft_erp>0.8</soft_erp>
+            <soft_erp>0.2</soft_erp>
             <kd>2500</kd>
             <kp>10</kp>
@@ -38,9 +38,6 @@
     <inertial>
       <origin xyz="0 0 0.01" rpy="0 0 0"/>
-      <mass value="0.1"/>
-      <inertia
-        ixx="0.01" ixy="0" ixz="0"
-        iyy="0.02" iyz="0"
-        izz="0.001"/>
+      <mass value="4.000000000" />
+      <inertia ixx="0.014166667" ixy="0.000000000" ixz="0.000000000" iyy="0.054166667" iyz="0.000000000" izz="0.066666667"/>
     </inertial>
   </link>
@@ -51,10 +48,10 @@
       </geometry>
     </collision>
-      <inertial>
-        <origin rpy="0 0 0" xyz="0 0 0" />
-        <mass value="0.000010000" />
-        <inertia ixx="0.000000010" ixy="0.000000000" ixz="0.000000000" iyy="0.000000010" iyz="0.000000000" izz="0.000000013"/>
-      </inertial>
-    </link>
+    <inertial>
+      <origin rpy="0 0 0" xyz="0 0 0" />
+      <mass value="1.000000000" />
+      <inertia ixx="0.001033333" ixy="0.000000000" ixz="0.000000000" iyy="0.001033333" iyz="0.000000000" izz="0.001250000"/>
+    </inertial>
+        </link>
   <link name="cylinder2">
     <collision>
@@ -63,10 +60,10 @@
       </geometry>
     </collision>
-      <inertial>
-        <origin rpy="0 0 0" xyz="0 0 0" />
-        <mass value="0.000010000" />
-        <inertia ixx="0.000000010" ixy="0.000000000" ixz="0.000000000" iyy="0.000000010" iyz="0.000000000" izz="0.000000013"/>
-      </inertial>
-    </link>
+    <inertial>
+      <origin rpy="0 0 0" xyz="0 0 0" />
+      <mass value="1.000000000" />
+      <inertia ixx="0.001033333" ixy="0.000000000" ixz="0.000000000" iyy="0.001033333" iyz="0.000000000" izz="0.001250000"/>
+    </inertial>
+        </link>
   <link name="head_plate">
     <visual>
@@ -155,4 +152,28 @@
   <origin xyz="0 -0.03 -0.01" rpy="0 0 0"/>
 </joint>
+<transmission name="motor1_trans">
+  <type>transmission_interface/SimpleTransmission</type>
+  <joint name="cylinder1_joint">
+    <hardwareInterface>EffortJointInterface</hardwareInterface>
+  </joint>
+  <actuator name="motor1_act">
+    <mechanicalReduction>50</mechanicalReduction>
+    <hardwareInterface>EffortJointInterface</hardwareInterface>
+  </actuator>
+</transmission>
+<transmission name="motor2_trans">
+  <type>transmission_interface/SimpleTransmission</type>
+  <joint name="cylinder2_joint">
+    <hardwareInterface>EffortJointInterface</hardwareInterface>
+  </joint>
+  <actuator name="motor1_act">
+    <mechanicalReduction>50</mechanicalReduction>
+    <hardwareInterface>EffortJointInterface</hardwareInterface>
+  </actuator>
+</transmission>
+<gazebo>
+  <plugin name="gazebo_ros_control" filename="libgazebo_ros_control.so">
+  </plugin>
+</gazebo>
 <gazebo reference="body">
   <material>Gazebo/Green</material>
@@ -172,5 +193,5 @@
         <max_vel>0.1</max_vel>
         <soft_cfm>0.8</soft_cfm>
-        <soft_erp>0.8</soft_erp>
+        <soft_erp>0.2</soft_erp>
         <kd>2500</kd>
         <kp>10</kp>
