Commit message: adding shuttle urdf model and collision simplified

File: aip_gazebo/models/cellule.urdf.xacro (robot description, xacro)
@@ -1,19 +1,20 @@
 <?xml version="1.0"?>
 <robot name="myfirst">
+  <link name="world"/>
   <link name="base_link"/>
   <link name="body">
     <visual>
       <geometry>
-        <mesh filename="file:////home/ugo/Desktop/Cours/3A/WORKSPACEROS/src/aip_gazebo/models/Cellule_lite.stl" scale="1 1 1"/>
+        <mesh filename="file:////home/ugo/Desktop/Cours/3A/WORKSPACEROS/src/aip_gazebo/models/v2/Cellule_empty.stl" scale="1 1 1"/>
       </geometry>
     </visual>
     <collision>
       <geometry>
-        <mesh filename="file:////home/ugo/Desktop/Cours/3A/WORKSPACEROS/src/aip_gazebo/models/Cellule_lite.stl" scale="1 1 1"/>
+        <mesh filename="file:///home/ugo/Desktop/Cours/3A/WORKSPACEROS/src/aip_gazebo/models/v2/Cellule_empty.stl" scale="1 1 1"/>
       </geometry>
     </collision>
     <inertial>
       <origin xyz="0 0 1" rpy="0 0 0"/>
-      <mass value="1"/>
+      <mass value="0.1"/>
       <inertia
         ixx="1.0" ixy="0.0" ixz="0.0"
@@ -22,4 +23,9 @@
     </inertial>
   </link>
+  <joint name="worldfixation" type="fixed">
+    <parent link="world"/>
+    <child link="base_link"/>
+    <origin xyz="0 0 0" rpy="0 0 0"/>
+</joint>
   <joint name="base_joint" type="fixed">
     <parent link="base_link"/>
@@ -27,8 +33,3 @@
     <origin xyz="0 0 0" rpy="0 0 0"/>
 </joint>
-<gazebo>
-  <plugin name="gazebo_ros_control" filename="libgazebo_ros_control.so">
-    <robotNamespace>/</robotNamespace>
-  </plugin>
-</gazebo>
 </robot>

File: aip_gazebo/models/shuttle.urdf.xacro (robot description, xacro)
@@ -5,19 +5,74 @@
     <visual>
       <geometry>
-        <mesh filename="file:////home/ugo/Desktop/Cours/3A/WORKSPACEROS/src/aip_gazebo/models/shuttle_parts/navette_body.stl" scale="0.03 0.03 0.03"/>
+        <mesh filename="file:////home/ugo/Desktop/Cours/3A/WORKSPACEROS/src/aip_gazebo/models/shuttle_parts/navette_body.stl" scale="0.04 0.04 0.04"/>
       </geometry>
     </visual>
     <collision>
+      <origin xyz="0.1 0 0.13" rpy="0 0 0"/>
       <geometry>
-        <mesh filename="file:////home/ugo/Desktop/Cours/3A/WORKSPACEROS/src/aip_gazebo/models/shuttle_parts/navette_body.stl" scale="0.03 0.03 0.03"/>
+        <box size="0.4 0.2 0.05" />
+      </geometry>
+      <surface>
+        <friction>
+          <ode>
+            <mu>0.5</mu>
+            <mu2>0.5</mu2>
+          </ode>
+        </friction>
+        <bounce>
+          <restitution_coefficient>0.01</restitution_coefficient>
+          <threshold>0.01</threshold>
+        </bounce>
+        <contact>
+          <ode>
+            <max_vel>0.1</max_vel>
+            <soft_cfm>0.8</soft_cfm>
+            <soft_erp>0.8</soft_erp>
+            <kd>2500</kd>
+            <kp>10</kp>
+            <min_depth>0.001</min_depth>
+          </ode>
+        </contact>
+      </surface>
+    </collision>
+    <inertial>
+      <origin xyz="0 0 0.01" rpy="0 0 0"/>
+      <mass value="0.1"/>
+      <inertia
+        ixx="0.01" ixy="0" ixz="0"
+        iyy="0.02" iyz="0"
+        izz="0.001"/>
+    </inertial>
+  </link>
+  <link name="cylinder1">
+    <collision>
+      <origin xyz="0 0 0.065" rpy="0 0 0"/>
+      <geometry>
+        <cylinder radius="0.05" length="0.07"/>
       </geometry>
     </collision>
     <inertial>
-      <origin xyz="0 0 1" rpy="0 0 0"/>
-      <mass value="1"/>
+      <origin xyz="0 0 0.01" rpy="0 0 0"/>
+      <mass value="0"/>
       <inertia
-        ixx="1.0" ixy="0.0" ixz="0.0"
-        iyy="1.0" iyz="0.0"
-        izz="1.0"/>
+        ixx="0.01" ixy="0" ixz="0"
+        iyy="0.02" iyz="0"
+        izz="0.001"/>
+    </inertial>
+  </link>
+  <link name="cylinder2">
+    <collision>
+      <origin xyz="0 0 0.065" rpy="0 0 0"/>
+      <geometry>
+        <cylinder radius="0.05" length="0.07"/>
+      </geometry>
+    </collision>
+    <inertial>
+      <origin xyz="0 0 0.01" rpy="0 0 0"/>
+      <mass value="0"/>
+      <inertia
+        ixx="0.01" ixy="0" ixz="0"
+        iyy="0.02" iyz="0"
+        izz="0.001"/>
     </inertial>
   </link>
@@ -27,8 +82,38 @@
     <origin xyz="0 0 0" rpy="0 0 0"/>
 </joint>
-<gazebo>
-  <plugin name="gazebo_ros_control" filename="libgazebo_ros_control.so">
-    <robotNamespace>/</robotNamespace>
-  </plugin>
+<joint name="cylinder1_joint" type="fixed">
+  <parent link="body"/>
+  <child link="cylinder1"/>
+  <origin xyz="0 0.07 0" rpy="0 0 0"/>
+</joint>
+<joint name="cylinder2_joint" type="fixed">
+  <parent link="body"/>
+  <child link="cylinder2"/>
+  <origin xyz="0 -0.07 0" rpy="0 0 0"/>
+</joint>
+<gazebo reference="body">
+  <material>Gazebo/Green</material>
+  <surface>
+    <friction>
+      <ode>
+        <mu>0.5</mu>
+        <mu2>0.5</mu2>
+      </ode>
+    </friction>
+    <bounce>
+      <restitution_coefficient>0.01</restitution_coefficient>
+      <threshold>0.01</threshold>
+    </bounce>
+    <contact>
+      <ode>
+        <max_vel>0.1</max_vel>
+        <soft_cfm>0.8</soft_cfm>
+        <soft_erp>0.8</soft_erp>
+        <kd>2500</kd>
+        <kp>10</kp>
+        <min_depth>0.001</min_depth>
+      </ode>
+    </contact>
+  </surface>
 </gazebo>
 </robot>

Commit message: changing path to relatives

File: aip_gazebo/models/cellule.urdf.xacro (robot description, xacro)
@@ -6,10 +6,10 @@
     <visual>
       <geometry>
-        <mesh filename="file:////home/ugo/Desktop/Cours/3A/WORKSPACEROS/src/aip_gazebo/models/v2/Cellule_empty.stl" scale="1 1 1"/>
+        <mesh filename="file://$(arg models_directory)/Cellule_lite.dae" scale="1 1 1"/>
       </geometry>
     </visual>
     <collision>
       <geometry>
-        <mesh filename="file:///home/ugo/Desktop/Cours/3A/WORKSPACEROS/src/aip_gazebo/models/v2/Cellule_empty.stl" scale="1 1 1"/>
+        <mesh filename="file://$(arg models_directory)/Cellule_lite.dae" scale="1 1 1"/>
       </geometry>
     </collision>

File: aip_gazebo/models/shuttle.urdf.xacro (robot description, xacro)
@@ -5,5 +5,5 @@
     <visual>
       <geometry>
-        <mesh filename="file:////home/ugo/Desktop/Cours/3A/WORKSPACEROS/src/aip_gazebo/models/shuttle_parts/navette_body.stl" scale="0.04 0.04 0.04"/>
+        <mesh filename="file://$(arg models_directory)/shuttle_parts/navette_body.stl" scale="0.04 0.04 0.04"/>
       </geometry>
     </visual>

Commit message: Ajout et fixation des aiguillages dans fichier URDF pour controle dynamique de la cellule dans futur

File: aip_gazebo/models/cellule.urdf.xacro (robot description, xacro)
@@ -1,4 +1,4 @@
 <?xml version="1.0"?>
-<robot name="myfirst">
+<robot name="cell">
   <link name="world"/>
   <link name="base_link"/>
@@ -6,10 +6,250 @@
     <visual>
       <geometry>
-        <mesh filename="file://$(arg models_directory)/Cellule_lite.dae" scale="1 1 1"/>
-      </geometry>
-    </visual>
-    <collision>
-      <geometry>
-        <mesh filename="file://$(arg models_directory)/Cellule_lite.dae" scale="1 1 1"/>
+        <mesh filename="file://$(arg models_directory)/v2/Cellule_empty.stl" scale="1 1 1"/>
+      </geometry>
+    </visual>
+    <collision>
+      <geometry>
+        <mesh filename="file://$(arg models_directory)/v2/Cellule_empty.stl" scale="1 1 1"/>
+      </geometry>
+    </collision>
+    <inertial>
+      <origin xyz="0 0 1" rpy="0 0 0"/>
+      <mass value="0.1"/>
+      <inertia
+        ixx="1.0" ixy="0.0" ixz="0.0"
+        iyy="1.0" iyz="0.0"
+        izz="1.0"/>
+    </inertial>
+  </link>
+  <link name="aig1">
+    <visual>
+      <geometry>
+        <mesh filename="file://$(arg models_directory)/v2/Aiguillage_centre.stl" scale="1.05 1.05 1"/>
+      </geometry>
+    </visual>
+    <collision>
+      <geometry>
+        <mesh filename="file://$(arg models_directory)/v2/Aiguillage_centre.stl" scale="1.05 1.05 1"/>
+      </geometry>
+    </collision>
+    <inertial>
+      <origin xyz="0 0 1" rpy="0 0 0"/>
+      <mass value="0.1"/>
+      <inertia
+        ixx="1.0" ixy="0.0" ixz="0.0"
+        iyy="1.0" iyz="0.0"
+        izz="1.0"/>
+    </inertial>
+  </link>
+  <link name="aig2">
+    <visual>
+      <geometry>
+        <mesh filename="file://$(arg models_directory)/v2/Aiguillage_centre.stl" scale="1.05 1.05 1"/>
+      </geometry>
+    </visual>
+    <collision>
+      <geometry>
+        <mesh filename="file://$(arg models_directory)/v2/Aiguillage_centre.stl" scale="1.05 1.05 1"/>
+      </geometry>
+    </collision>
+    <inertial>
+      <origin xyz="0 0 1" rpy="0 0 0"/>
+      <mass value="0.1"/>
+      <inertia
+        ixx="1.0" ixy="0.0" ixz="0.0"
+        iyy="1.0" iyz="0.0"
+        izz="1.0"/>
+    </inertial>
+  </link>
+  <link name="aig3">
+    <visual>
+      <geometry>
+        <mesh filename="file://$(arg models_directory)/v2/Aiguillage_centre.stl" scale="1.05 1.05 1"/>
+      </geometry>
+    </visual>
+    <collision>
+      <geometry>
+        <mesh filename="file://$(arg models_directory)/v2/Aiguillage_centre.stl" scale="1.05 1.05 1"/>
+      </geometry>
+    </collision>
+    <inertial>
+      <origin xyz="0 0 1" rpy="0 0 0"/>
+      <mass value="0.1"/>
+      <inertia
+        ixx="1.0" ixy="0.0" ixz="0.0"
+        iyy="1.0" iyz="0.0"
+        izz="1.0"/>
+    </inertial>
+  </link>
+  <link name="aig4">
+    <visual>
+      <geometry>
+        <mesh filename="file://$(arg models_directory)/v2/Aiguillage_centre.stl" scale="1.05 1.05 1"/>
+      </geometry>
+    </visual>
+    <collision>
+      <geometry>
+        <mesh filename="file://$(arg models_directory)/v2/Aiguillage_centre.stl" scale="1.05 1.05 1"/>
+      </geometry>
+    </collision>
+    <inertial>
+      <origin xyz="0 0 1" rpy="0 0 0"/>
+      <mass value="0.1"/>
+      <inertia
+        ixx="1.0" ixy="0.0" ixz="0.0"
+        iyy="1.0" iyz="0.0"
+        izz="1.0"/>
+    </inertial>
+  </link>
+  <link name="aig5">
+    <visual>
+      <geometry>
+        <mesh filename="file://$(arg models_directory)/v2/Aiguillage_centre.stl" scale="1.05 1.05 1"/>
+      </geometry>
+    </visual>
+    <collision>
+      <geometry>
+        <mesh filename="file://$(arg models_directory)/v2/Aiguillage_centre.stl" scale="1.05 1.05 1"/>
+      </geometry>
+    </collision>
+    <inertial>
+      <origin xyz="0 0 1" rpy="0 0 0"/>
+      <mass value="0.1"/>
+      <inertia
+        ixx="1.0" ixy="0.0" ixz="0.0"
+        iyy="1.0" iyz="0.0"
+        izz="1.0"/>
+    </inertial>
+  </link>
+  <link name="aig6">
+    <visual>
+      <geometry>
+        <mesh filename="file://$(arg models_directory)/v2/Aiguillage_centre.stl" scale="1.05 1.05 1"/>
+      </geometry>
+    </visual>
+    <collision>
+      <geometry>
+        <mesh filename="file://$(arg models_directory)/v2/Aiguillage_centre.stl" scale="1.05 1.05 1"/>
+      </geometry>
+    </collision>
+    <inertial>
+      <origin xyz="0 0 1" rpy="0 0 0"/>
+      <mass value="0.1"/>
+      <inertia
+        ixx="1.0" ixy="0.0" ixz="0.0"
+        iyy="1.0" iyz="0.0"
+        izz="1.0"/>
+    </inertial>
+  </link>
+  <link name="aig7">
+    <visual>
+      <geometry>
+        <mesh filename="file://$(arg models_directory)/v2/Aiguillage_centre.stl" scale="1.05 1.05 1"/>
+      </geometry>
+    </visual>
+    <collision>
+      <geometry>
+        <mesh filename="file://$(arg models_directory)/v2/Aiguillage_centre.stl" scale="1.05 1.05 1"/>
+      </geometry>
+    </collision>
+    <inertial>
+      <origin xyz="0 0 1" rpy="0 0 0"/>
+      <mass value="0.1"/>
+      <inertia
+        ixx="1.0" ixy="0.0" ixz="0.0"
+        iyy="1.0" iyz="0.0"
+        izz="1.0"/>
+    </inertial>
+  </link>
+  <link name="aig8">
+    <visual>
+      <geometry>
+        <mesh filename="file://$(arg models_directory)/v2/Aiguillage_centre.stl" scale="1.05 1.05 1"/>
+      </geometry>
+    </visual>
+    <collision>
+      <geometry>
+        <mesh filename="file://$(arg models_directory)/v2/Aiguillage_centre.stl" scale="1.05 1.05 1"/>
+      </geometry>
+    </collision>
+    <inertial>
+      <origin xyz="0 0 1" rpy="0 0 0"/>
+      <mass value="0.1"/>
+      <inertia
+        ixx="1.0" ixy="0.0" ixz="0.0"
+        iyy="1.0" iyz="0.0"
+        izz="1.0"/>
+    </inertial>
+  </link>
+  <link name="aig9">
+    <visual>
+      <geometry>
+        <mesh filename="file://$(arg models_directory)/v2/Aiguillage_centre.stl" scale="1.05 1.05 1"/>
+      </geometry>
+    </visual>
+    <collision>
+      <geometry>
+        <mesh filename="file://$(arg models_directory)/v2/Aiguillage_centre.stl" scale="1.05 1.05 1"/>
+      </geometry>
+    </collision>
+    <inertial>
+      <origin xyz="0 0 1" rpy="0 0 0"/>
+      <mass value="0.1"/>
+      <inertia
+        ixx="1.0" ixy="0.0" ixz="0.0"
+        iyy="1.0" iyz="0.0"
+        izz="1.0"/>
+    </inertial>
+  </link>
+  <link name="aig10">
+    <visual>
+      <geometry>
+        <mesh filename="file://$(arg models_directory)/v2/Aiguillage_centre.stl" scale="1.05 1.05 1"/>
+      </geometry>
+    </visual>
+    <collision>
+      <geometry>
+        <mesh filename="file://$(arg models_directory)/v2/Aiguillage_centre.stl" scale="1.05 1.05 1"/>
+      </geometry>
+    </collision>
+    <inertial>
+      <origin xyz="0 0 1" rpy="0 0 0"/>
+      <mass value="0.1"/>
+      <inertia
+        ixx="1.0" ixy="0.0" ixz="0.0"
+        iyy="1.0" iyz="0.0"
+        izz="1.0"/>
+    </inertial>
+  </link>
+  <link name="aig11">
+    <visual>
+      <geometry>
+        <mesh filename="file://$(arg models_directory)/v2/Aiguillage_centre.stl" scale="1.05 1.05 1"/>
+      </geometry>
+    </visual>
+    <collision>
+      <geometry>
+        <mesh filename="file://$(arg models_directory)/v2/Aiguillage_centre.stl" scale="1.05 1.05 1"/>
+      </geometry>
+    </collision>
+    <inertial>
+      <origin xyz="0 0 1" rpy="0 0 0"/>
+      <mass value="0.1"/>
+      <inertia
+        ixx="1.0" ixy="0.0" ixz="0.0"
+        iyy="1.0" iyz="0.0"
+        izz="1.0"/>
+    </inertial>
+  </link>
+  <link name="aig12">
+    <visual>
+      <geometry>
+        <mesh filename="file://$(arg models_directory)/v2/Aiguillage_centre.stl" scale="1.05 1.05 1"/>
+      </geometry>
+    </visual>
+    <collision>
+      <geometry>
+        <mesh filename="file://$(arg models_directory)/v2/Aiguillage_centre.stl" scale="1.05 1.05 1"/>
       </geometry>
     </collision>
@@ -28,4 +268,64 @@
     <origin xyz="0 0 0" rpy="0 0 0"/>
 </joint>
+<joint name="aig1_joint" type="fixed">
+  <parent link="base_link"/>
+  <child link="aig1"/>
+  <origin xyz="-2.995740 -2.589235 0.703549" rpy="0 0 0"/>
+</joint>
+<joint name="aig2_joint" type="fixed">
+  <parent link="base_link"/>
+  <child link="aig2"/>
+  <origin xyz="-1.530460 -2.495351 0.703549" rpy="0 0 -0.522816"/>
+</joint>
+<joint name="aig3_joint" type="fixed">
+  <parent link="base_link"/>
+  <child link="aig3"/>
+  <origin xyz="-1.531780 -3.242463 0.703549 " rpy="0 0 0.522816"/>
+</joint>
+<joint name="aig4_joint" type="fixed">
+  <parent link="base_link"/>
+  <child link="aig4"/>
+  <origin xyz="-2.996613 -3.148634 0.703549" rpy="0 0 0"/>
+</joint>
+<joint name="aig5_joint" type="fixed">
+  <parent link="base_link"/>
+  <child link="aig5"/>
+  <origin xyz="-0.969881 -2.682101 0.703549" rpy="0 0 -1.564166"/>
+</joint>
+<joint name="aig6_joint" type="fixed">
+  <parent link="base_link"/>
+  <child link="aig6"/>
+  <origin xyz="-0.970147 -3.054364 0.703549" rpy="0 0 1.557541"/>
+</joint>
+<joint name="aig7_joint" type="fixed">
+  <parent link="base_link"/>
+  <child link="aig7"/>
+  <origin xyz="1.150706 -2.495223 0.703549" rpy="0 0 -0.522816"/>
+</joint>
+<joint name="aig8_joint" type="fixed">
+  <parent link="base_link"/>
+  <child link="aig8"/>
+  <origin xyz="2.615560 -2.589317 0.703549" rpy="0 0 1.051898"/>
+</joint>
+<joint name="aig9_joint" type="fixed">
+  <parent link="base_link"/>
+  <child link="aig9"/>
+  <origin xyz="2.616508 -3.147677 0.703549" rpy="0 0 3.126283"/>
+</joint>
+<joint name="aig10_joint" type="fixed">
+  <parent link="base_link"/>
+  <child link="aig10"/>
+  <origin xyz="1.147324 -3.242931 0.703549" rpy="0 0 0.522816"/>
+</joint>
+<joint name="aig11_joint" type="fixed">
+  <parent link="base_link"/>
+  <child link="aig11"/>
+  <origin xyz="0.590738 -2.682604 0.703549" rpy="0 0 -1.564169"/>
+</joint>
+<joint name="aig12_joint" type="fixed">
+  <parent link="base_link"/>
+  <child link="aig12"/>
+  <origin xyz="0.591956 -3.055061 0.703549" rpy="0 0 1.557539"/>
+</joint>
   <joint name="base_joint" type="fixed">
     <parent link="base_link"/>

File: aip_gazebo/models/shuttle.urdf.xacro (robot description, xacro)
@@ -1,4 +1,4 @@
 <?xml version="1.0"?>
-<robot name="myfirst">
+<robot name="shuttle">
   <link name="base_link"/>
   <link name="body">
