Commit message: changing friction + modeling back joint + adaptation of the cell

File: aip_gazebo/models/cellule.urdf.xacro (robot description, xacro)
@@ -301,5 +301,5 @@
   <parent link="base_link"/>
   <child link="aig7"/>
-  <origin xyz="1.150706 -2.495223 0.703549" rpy="0 0 -0.522816"/>
+  <origin xyz="1.150706 -2.495223 0.703549" rpy="0 0 1.58"/>
 </joint>
 <joint name="aig8_joint" type="fixed">
@@ -311,10 +311,10 @@
   <parent link="base_link"/>
   <child link="aig9"/>
-  <origin xyz="2.616508 -3.147677 0.703549" rpy="0 0 3.126283"/>
+  <origin xyz="2.616508 -3.147677 0.703549" rpy="0 0 5.25"/>
 </joint>
 <joint name="aig10_joint" type="fixed">
   <parent link="base_link"/>
   <child link="aig10"/>
-  <origin xyz="1.147324 -3.242931 0.703549" rpy="0 0 0.522816"/>
+  <origin xyz="1.147324 -3.242931 0.703549" rpy="0 0 -1.564169"/>
 </joint>
 <joint name="aig11_joint" type="fixed">

File: aip_gazebo/models/shuttle.urdf.xacro (robot description, xacro)
@@ -4,18 +4,20 @@
   <link name="body">
     <visual>
-      <geometry>
-        <mesh filename="file://$(arg models_directory)/shuttle_parts/navette_body.stl" scale="0.04 0.04 0.04"/>
-      </geometry>
-    </visual>
-    <collision>
       <origin xyz="0.1 0 0.13" rpy="0 0 0"/>
       <geometry>
         <box size="0.4 0.2 0.05" />
-      </geometry>
-      <surface>
-        <friction>
-          <ode>
-            <mu>0.5</mu>
-            <mu2>0.5</mu2>
+        <!--mesh filename="file://$(arg models_directory)/shuttle_parts/navette_body.stl" scale="0.04 0.04 0.04"/-->
+      </geometry>
+    </visual>
+    <collision>
+      <origin xyz="0.1 0 0.13" rpy="0 0 0"/>
+      <geometry>
+        <box size="0.4 0.2 0.05" />
+      </geometry>
+      <surface>
+        <friction>
+          <ode>
+            <mu>0.01</mu>
+            <mu2>0.01</mu2>
           </ode>
         </friction>
@@ -32,19 +34,76 @@
             <kp>10</kp>
             <min_depth>0.001</min_depth>
-          </ode>
+          </ode>C:\home\ugo\Desktop\Cours\3A\WORKSPACEROS> ^C
+          C:\home\ugo\Desktop\Cours\3A\WORKSPACEROS> ^C
         </contact>
       </surface>
     </collision>
     <inertial>
-      <origin xyz="0 0 0.01" rpy="0 0 0"/>
+      <origin xyz="0.15 0 0.12" rpy="0 0 0"/>
       <mass value="4.000000000" />
       <inertia ixx="0.014166667" ixy="0.000000000" ixz="0.000000000" iyy="0.054166667" iyz="0.000000000" izz="0.066666667"/>
     </inertial>
   </link>
+  <link name="ski">
+    <visual>
+      <geometry>
+        <box size="0.06 0.1 0.01" />
+        <!--mesh filename="file://$(arg models_directory)/shuttle_parts/navette_body.stl" scale="0.04 0.04 0.04"/-->
+      </geometry>
+    </visual>
+    <collision>
+      <geometry>
+        <box size="0.06 0.1 0.01" />
+      </geometry>
+      <surface>
+        <friction>
+          <ode>
+            <mu>0.01</mu>
+            <mu2>0.01</mu2>
+          </ode>
+        </friction>
+      </surface>
+    </collision>
+    <inertial>
+      <origin rpy="0 0 0" xyz="0 0 0" />
+      <mass value="0.200000000" />
+      <inertia ixx="0.000168333" ixy="0.000000000" ixz="0.000000000" iyy="0.000061667" iyz="0.000000000" izz="0.000226667"/>
+    </inertial>
+  </link>
+  <link name="tail_plate">
+    <visual>
+      <geometry>
+        <box size="0.03 0.1 0.01" />
+      </geometry>
+    </visual>
+    <collision>
+      <geometry>
+        <box size="0.03 0.05 0.01" />
+      </geometry>
+    </collision>
+    <inertial>
+      <origin rpy="0 0 0" xyz="0 0 0" />
+      <mass value="0.300000000" />
+      <inertia ixx="0.000065000" ixy="0.000000000" ixz="0.000000000" iyy="0.000025000" iyz="0.000000000" izz="0.000085000"/>
+    </inertial>
+  </link>
   <link name="cylinder1">
-    <collision>
-      <geometry>
-        <cylinder radius="0.05" length="0.07"/>
-      </geometry>
+    <visual>
+      <geometry>
+        <cylinder radius="0.055" length="0.04"/>
+      </geometry>
+    </visual>
+    <collision>
+      <geometry>
+        <cylinder radius="0.055" length="0.04"/>
+      </geometry>
+      <surface>
+        <friction>
+          <ode>
+            <mu>0.9</mu>
+            <mu2>0.9</mu2>
+          </ode>
+        </friction>
+      </surface>
     </collision>
     <inertial>
@@ -55,7 +114,12 @@
         </link>
   <link name="cylinder2">
-    <collision>
-      <geometry>
-        <cylinder radius="0.05" length="0.07"/>
+    <visual>
+      <geometry>
+        <cylinder radius="0.055" length="0.04"/>
+      </geometry>
+    </visual>
+    <collision>
+      <geometry>
+        <cylinder radius="0.055" length="0.04"/>
       </geometry>
     </collision>
@@ -76,45 +140,69 @@
         <box size="0.03 0.05 0.01" />
       </geometry>
-    </collision>
-    <inertial>
-      <origin rpy="0 0 0" xyz="0 0 0" />
-      <mass value="0.000010000" />
-      <inertia ixx="0.000000002" ixy="0.000000000" ixz="0.000000000" iyy="0.000000001" iyz="0.000000000" izz="0.000000003"/>
+      <surface>
+        <friction>
+          <ode>
+            <mu>0.01</mu>
+            <mu2>0.01</mu2>
+          </ode>
+        </friction>
+      </surface>
+    </collision>
+    <inertial>
+      <origin rpy="0 0 0" xyz="0 0 0" />
+      <mass value="0.300000000" />
+      <inertia ixx="0.000065000" ixy="0.000000000" ixz="0.000000000" iyy="0.000025000" iyz="0.000000000" izz="0.000085000"/>
+    </inertial>
+  </link>
+  <link name="free_wheel_1">
+    <visual>
+      <geometry>
+        <cylinder radius="0.02" length="0.1"/>
+      </geometry>
+    </visual>
+    <collision>
+      <geometry>
+        <cylinder radius="0.02" length="0.1"/>
+      </geometry>
+      <surface>
+        <friction>
+          <ode>
+            <mu>0.01</mu>
+            <mu2>0.01</mu2>
+          </ode>
+        </friction>
+      </surface>
+    </collision>
+    <inertial>
+      <origin rpy="0 0 0" xyz="0 0 0" />
+      <mass value="0.500000000" />
+      <inertia ixx="0.000429167" ixy="0.000000000" ixz="0.000000000" iyy="0.000429167" iyz="0.000000000" izz="0.000025000"/>
+    </inertial>
+          </link>
+  <link name="free_wheel_2">
+    <visual>
+      <geometry>
+        <cylinder radius="0.02" length="0.1"/>
+      </geometry>
+    </visual>
+    <collision>
+      <geometry>
+        <cylinder radius="0.02" length="0.1"/>
+      </geometry>
+      <surface>
+        <friction>
+          <ode>
+            <mu>0.01</mu>
+            <mu2>0.01</mu2>
+          </ode>
+        </friction>
+      </surface>
+    </collision>
+    <inertial>
+      <origin rpy="0 0 0" xyz="0 0 0" />
+      <mass value="0.500000000" />
+      <inertia ixx="0.000429167" ixy="0.000000000" ixz="0.000000000" iyy="0.000429167" iyz="0.000000000" izz="0.000025000"/>
     </inertial>
         </link>
-  <link name="free_wheel_1">
-    <visual>
-      <geometry>
-        <cylinder radius="0.01" length="0.02"/>
-      </geometry>
-    </visual>
-    <collision>
-      <geometry>
-        <cylinder radius="0.01" length="0.02"/>
-      </geometry>
-    </collision>
-    <inertial>
-      <origin rpy="0 0 0" xyz="0 0 0" />
-      <mass value="0.000010000" />
-      <inertia ixx="0.000000001" ixy="0.000000000" ixz="0.000000000" iyy="0.000000001" iyz="0.000000000" izz="0.000000001"/>
-    </inertial>
-      </link>
-  <link name="free_wheel_2">
-    <visual>
-      <geometry>
-        <cylinder radius="0.01" length="0.02"/>
-      </geometry>
-    </visual>
-    <collision>
-      <geometry>
-        <cylinder radius="0.01" length="0.02"/>
-      </geometry>
-    </collision>
-    <inertial>
-      <origin rpy="0 0 0" xyz="0 0 0" />
-      <mass value="0.000010000" />
-      <inertia ixx="0.000000001" ixy="0.000000000" ixz="0.000000000" iyy="0.000000001" iyz="0.000000000" izz="0.000000001"/>
-    </inertial>
-    </link>
 <joint name="base_joint" type="fixed">
   <parent link="base_link"/>
@@ -122,27 +210,38 @@
   <origin xyz="0 0 0" rpy="0 0 0"/>
 </joint>
+<joint name="ski_joint" type="fixed">
+  <parent link="body"/>
+  <child link="ski"/>
+  <origin xyz="0.32 0 0.11" rpy="0 -0.5 0"/>
+</joint>
+<joint name="tail_plate_joint" type="continuous">
+  <parent link="body"/>
+  <child link="tail_plate"/>
+  <axis xyz="0 0 1"/>
+  <origin xyz="0 0 0.12" rpy="0 0 0"/>
+</joint>
 <joint name="cylinder1_joint" type="continuous">
-<parent link="body"/>
+<parent link="tail_plate"/>
 <child link="cylinder1"/>
 <axis xyz="0 0 1"/>
-<origin xyz="0 0.07 0.065" rpy="0 0 0"/>
+<origin xyz="0 0.07 -0.07" rpy="0.0 0 0"/>
 </joint>
 <joint name="cylinder2_joint" type="continuous">
-<parent link="body"/>
+<parent link="tail_plate"/>
 <child link="cylinder2"/>
 <axis xyz="0 0 1"/>
-<origin xyz="0 -0.07 0.065" rpy="0 0 0"/>
-</joint>
-<joint name="free_plate" type="fixed">
+<origin xyz="0 -0.07 -0.07" rpy="0.0 0 0"/>
+</joint>
+<joint name="free_plate" type="continuous">
   <parent link="body"/>
   <child link="head_plate"/>
   <axis xyz="0 0 1"/>
-  <origin xyz="0.3 0 0.11" rpy="0 0 0"/>
-</joint>
-<joint name="free_wheel_1_joint" type="fixed">
+  <origin xyz="0.3 0 0.12" rpy="0 0 0"/>
+</joint>
+<joint name="free_wheel_1_joint" type="continuous">
   <parent link="head_plate"/>
   <child link="free_wheel_1"/>
   <axis xyz="0 0 1"/>
-  <origin xyz="0 0.03 -0.01" rpy="0 0 0"/>
+  <origin xyz="0 0.05 -0.05" rpy="0 0 0"/>
 </joint>
 <joint name="free_wheel_2_joint" type="continuous">
@@ -150,5 +249,5 @@
   <child link="free_wheel_2"/>
   <axis xyz="0 0 1"/>
-  <origin xyz="0 -0.03 -0.01" rpy="0 0 0"/>
+  <origin xyz="0 -0.05 -0.05" rpy="0 0 0"/>
 </joint>
 <transmission name="motor1_trans">
